Commit message: template code for inverse kinematics/dynamics using pinocchio

File: data/urdf/solo12_test.urdf (robot description, URDF)
Before this commit: robot solo, 17 links, 16 joints
Links:
- link base_link: mass 2.5 -> 1.16115091

File: data/urdf/solo12_update.urdf (robot description, URDF)
Before this commit: robot solo, 17 links, 16 joints
Links:
- link FL_FOOT: geometry collision mesh filename=package://example-robot-data/robots/solo_description/meshes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; visual mesh filename=package://example-robot-data/robots/solo_description/meshes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
- link FL_LOWER_LEG: geometry collision mesh filename=package://example-robot-data/robots/solo_description/meshes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; visual mesh filename=package://example-robot-data/robots/solo_description/meshes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
- link FL_SHOULDER: geometry collision mesh filename=package://example-robot-data/robots/solo_description/meshes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; visual mesh filename=package://example-robot-data/robots/solo_description/meshes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
- link FL_UPPER_LEG: geometry collision mesh filename=package://example-robot-data/robots/solo_description/meshes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; visual mesh filename=package://example-robot-data/robots/solo_description/meshes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
- link FR_FOOT: geometry collision mesh filename=package://example-robot-data/robots/solo_description/meshes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; visual mesh filename=package://example-robot-data/robots/solo_description/meshes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
- link FR_LOWER_LEG: geometry collision mesh filename=package://example-robot-data/robots/solo_description/meshes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; visual mesh filename=package://example-robot-data/robots/solo_description/meshes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
- link FR_SHOULDER: geometry collision mesh filename=package://example-robot-data/robots/solo_description/meshes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; visual mesh filename=package://example-robot-data/robots/solo_description/meshes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
- link FR_UPPER_LEG: geometry collision mesh filename=package://example-robot-data/robots/solo_description/meshes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; visual mesh filename=package://example-robot-data/robots/solo_description/meshes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
- link HL_FOOT: geometry collision mesh filename=package://example-robot-data/robots/solo_description/meshes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; visual mesh filename=package://example-robot-data/robots/solo_description/meshes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
- link HL_LOWER_LEG: geometry collision mesh filename=package://example-robot-data/robots/solo_description/meshes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; visual mesh filename=package://example-robot-data/robots/solo_description/meshes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
- link HL_SHOULDER: geometry collision mesh filename=package://example-robot-data/robots/solo_description/meshes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; visual mesh filename=package://example-robot-data/robots/solo_description/meshes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
- link HL_UPPER_LEG: geometry collision mesh filename=package://example-robot-data/robots/solo_description/meshes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; visual mesh filename=package://example-robot-data/robots/solo_description/meshes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
- link HR_FOOT: geometry collision mesh filename=package://example-robot-data/robots/solo_description/meshes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; visual mesh filename=package://example-robot-data/robots/solo_description/meshes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
- link HR_LOWER_LEG: geometry collision mesh filename=package://example-robot-data/robots/solo_description/meshes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; visual mesh filename=package://example-robot-data/robots/solo_description/meshes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
- link HR_SHOULDER: geometry collision mesh filename=package://example-robot-data/robots/solo_description/meshes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; visual mesh filename=package://example-robot-data/robots/solo_description/meshes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
- link HR_UPPER_LEG: geometry collision mesh filename=package://example-robot-data/robots/solo_description/meshes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; visual mesh filename=package://example-robot-data/robots/solo_description/meshes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
- link base_link: mass 1.5 -> 1.16115091; geometry collision mesh filename=package://example-robot-data/robots/solo_description/meshes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; visual mesh filename=package://example-robot-data/robots/solo_description/meshes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
Joints:
- joint FL_HAA: origin xyz=0.1946 0.08750000000000001 0 rpy=0 0 0 -> xyz=0.1946 0.0875 0 rpy=0 0 0
- joint FL_KFE: origin xyz=0 0.037450000000000004 -0.16 rpy=0 0 0 -> xyz=0 0.03745 -0.16 rpy=0 0 0
- joint FR_HAA: origin xyz=0.1946 -0.08750000000000001 0 rpy=0 0 0 -> xyz=0.1946 -0.0875 0 rpy=0 0 0
- joint FR_KFE: origin xyz=0 -0.037450000000000004 -0.16 rpy=0 0 0 -> xyz=0 -0.03745 -0.16 rpy=0 0 0
- joint HL_HAA: origin xyz=-0.1946 0.08750000000000001 0 rpy=0 0 0 -> xyz=-0.1946 0.0875 0 rpy=0 0 0
- joint HL_KFE: origin xyz=0 0.037450000000000004 -0.16 rpy=0 0 0 -> xyz=0 0.03745 -0.16 rpy=0 0 0
- joint HR_HAA: origin xyz=-0.1946 -0.08750000000000001 0 rpy=0 0 0 -> xyz=-0.1946 -0.0875 0 rpy=0 0 0
- joint HR_KFE: origin xyz=0 -0.037450000000000004 -0.16 rpy=0 0 0 -> xyz=0 -0.03745 -0.16 rpy=0 0 0
