Commit message: walking example works, need to implement torque based control and fix coeff in bezier curve

File: data/urdf/solo12.urdf (robot description, URDF)
Before this commit: robot solo, 17 links, 16 joints
Links:
- link base_link: mass 1.16115091 -> 100.16115091

Commit message: working simple simulation env

File: data/urdf/solo12.urdf (robot description, URDF)
Before this commit: robot solo, 17 links, 16 joints
Links:
- link base_link: mass 100.16115091 -> 100

Commit message: updated to timestep in simulation so it runs more like real time

File: data/urdf/solo12.urdf (robot description, URDF)
Before this commit: robot solo, 17 links, 16 joints
Links:
- link base_link: mass 100 -> 10

Commit message: init stance is implemented with keyboard press

File: data/urdf/solo12.urdf (robot description, URDF)
Before this commit: robot solo, 17 links, 16 joints
Links:
- link base_link: mass 10 -> 1.00

Commit message: flag switches work

File: data/urdf/solo12.urdf (robot description, URDF)
Before this commit: robot solo, 17 links, 16 joints
Links:
- link base_link: mass 1.00 -> 1.0

Commit message: fixes to trajectory collection script

File: data/urdf/solo12.urdf (robot description, URDF)
Before this commit: robot solo, 17 links, 16 joints
Links:
- link base_link: mass 1.0 -> 1.5

Commit message: update

File: data/urdf/solo12.urdf (robot description, URDF)
Before this commit: robot solo, 17 links, 16 joints
Links:
- link base_link: mass 1.5 -> 1.16115091

Commit message: bug fixes

File: data/urdf/solo12.urdf (robot description, URDF)
Before this commit: robot solo, 17 links, 16 joints
Links:
- link base_link: mass 1.16115091 -> 1.5

Commit message: fixed stance bug

File: data/urdf/solo12.urdf (robot description, URDF)
Before this commit: robot solo, 17 links, 16 joints
Links:
- link base_link: mass 1.5 -> 2.5
